File: hardware/nevil_sbc_rev0/nevil_sbc_rev0.kicad_sch (KiCad schematic)
At the start: 35 parts

Commit message: Updating schematics
Parts:
- added U?: ATtiny84-20P, Package_DIP:DIP-14_W7.62mm, symbol MCU_Microchip_ATtiny:ATtiny84-20P
Other:
- added sheet Peripherals (peripherals.kicad_sch)
Changed lines of the file:
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@@
     (pin "1")
+  )
+  (symbol (lib_id "MCU_Microchip_ATtiny:ATtiny84-20P") (at -129.54 -15.24 0) (unit 1)
+    (in_bom yes) (on_board yes) (fields_autoplaced)
+    (property "Reference" "U?" (id 0) (at -142.24 -16.5101 0)
+      (effects (font (size 1.27 1.27)) (justify right))
+    )
+    (property "Value" "ATtiny84-20P" (id 1) (at -142.24 -13.9701 0)
+      (effects (font (size 1.27 1.27)) (justify right))
+    )
+    (property "Footprint" "Package_DIP:DIP-14_W7.62mm" (id 2) (at -129.54 -15.24 0)
+      (effects (font (size 1.27 1.27) italic) hide)
+    )
+    (property "Datasheet" "http://ww1.microchip.com/downloads/en/DeviceDoc/doc8006.pdf" (id 3) (at -129.54 -15.24 0)
+      (effects (font (size 1.27 1.27)) hide)
+    )
+    (pin "1")
+    (pin "10")
+    (pin "11")
+    (pin "12")
+    (pin "13")
+    (pin "14")
+    (pin "2")
+    (pin "3")
+    (pin "4")
+    (pin "5")
+    (pin "6")
+    (pin "7")
+    (pin "8")
+    (pin "9")
   )
   (symbol (lib_id "65xx:W65C22SxP") (at -33.02 133.35 0) (unit 1)
@@
     (pin "2")
   )
+  (sheet (at 204.47 41.91) (size 22.86 16.51) (fields_autoplaced)
+    (stroke (width 0.1524) (type solid) (color 0 0 0 0))
+    (fill (color 0 0 0 0.0000))
+    (property "Sheet name" "Peripherals" (id 0) (at 204.47 41.1984 0)
+      (effects (font (size 1.27 1.27)) (justify left bottom))
+    )
+    (property "Sheet file" "peripherals.kicad_sch" (id 1) (at 204.47 59.0046 0)
+      (effects (font (size 1.27 1.27)) (justify left top))
+    )
+  )
   (sheet_instances
     (path "/" (page "1"))
+    (path "/47e5f244-199c-483d-9129-db89de2f9ca8" (page "2"))
   )
   (symbol_instances
@@
       (reference "C?") (unit 1) (value "0.1uF") (footprint "")
     )
+    (path "/47e5f244-199c-483d-9129-db89de2f9ca8/e348be46-6574-4ba9-9966-1c4b0473ed8c"
+      (reference "C?") (unit 1) (value "0.1uF") (footprint "")
+    )
     (path "/e8e20204-7e9c-48ca-8281-0e72ee50389b"
       (reference "C?") (unit 1) (value "1000uF") (footprint "")
     )
+    (path "/47e5f244-199c-483d-9129-db89de2f9ca8/ea7ac4dc-6ee8-44f6-a134-d247f2e45705"
+      (reference "C?") (unit 1) (value "1000uF") (footprint "")
+    )
     (path "/156bb2ef-c9f6-4267-a4cd-6be6db8068ad"
       (reference "J?") (unit 1) (value "Jack-DC") (footprint "")
@@
       (reference "R?") (unit 1) (value "1K") (footprint "")
     )
+    (path "/47e5f244-199c-483d-9129-db89de2f9ca8/bc2118bf-1e52-473f-86e1-9d70f2c0a7cd"
+      (reference "R?") (unit 1) (value "R_Small") (footprint "")
+    )
     (path "/c3b26662-b508-402c-a774-e93a5a47c493"
       (reference "R?") (unit 1) (value "1K") (footprint "")
@@
       (reference "SW?") (unit 1) (value "RESET") (footprint "")
     )
+    (path "/47e5f244-199c-483d-9129-db89de2f9ca8/047c69ed-8118-47c6-85be-ba76a79ec70c"
+      (reference "U?") (unit 1) (value "74LS245") (footprint "Package_DIP:DIP-20_W7.62mm_Socket_LongPads")
+    )
     (path "/0c0b8495-ef12-4548-89d3-aaad0eac09b6"
       (reference "U?") (unit 1) (value "CY62256-70PC") (footprint "Package_DIP:DIP-28_W15.24mm")
@@
       (reference "U?") (unit 1) (value "NE555D") (footprint "Package_SO:SOIC-8_3.9x4.9mm_P1.27mm")
     )
+    (path "/47e5f244-199c-483d-9129-db89de2f9ca8/396edc42-b52d-4806-b6ca-28b3204b9bb1"
+      (reference "U?") (unit 1) (value "74HC00") (footprint "")
+    )
+    (path "/47e5f244-199c-483d-9129-db89de2f9ca8/53559ba4-1e5c-4536-8366-eb67a1567afc"
+      (reference "U?") (unit 1) (value "28C256") (footprint "Package_DIP:DIP-28_W15.24mm_Socket_LongPads")
+    )
     (path "/60d9d493-08f0-4352-abaa-44052742e635"
       (reference "U?") (unit 1) (value "74LS245") (footprint "Package_DIP:DIP-20_W7.62mm_Socket_LongPads")
@@
       (reference "U?") (unit 1) (value "28C256") (footprint "Package_DIP:DIP-28_W15.24mm_Socket_LongPads")
     )
+    (path "/47e5f244-199c-483d-9129-db89de2f9ca8/858dcf5b-9c9c-4827-bc2c-8fe00084c5e6"
+      (reference "U?") (unit 1) (value "ATtiny84-20P") (footprint "Package_DIP:DIP-14_W7.62mm")
+    )
+    (path "/47e5f244-199c-483d-9129-db89de2f9ca8/88d32f5a-4188-43e2-ae0a-3c1a0d500750"
+      (reference "U?") (unit 1) (value "W65C22SxP") (footprint "")
+    )
+    (path "/47e5f244-199c-483d-9129-db89de2f9ca8/97f37e71-f1d7-46e7-9231-dab8f2eeb161"
+      (reference "U?") (unit 1) (value "W65C22SxP") (footprint "Package_DIP:DIP-40_W15.24mm_Socket_LongPads")
+    )
     (path "/9b75079b-c2c4-477e-8c55-ef0d0343d3d5"
       (reference "U?") (unit 1) (value "74HC00") (footprint "")
@@
       (reference "U?") (unit 1) (value "W65C22SxP") (footprint "Package_DIP:DIP-40_W15.24mm_Socket_LongPads")
     )
+    (path "/47e5f244-199c-483d-9129-db89de2f9ca8/c60c38c8-41e7-498c-8cfa-1a05866f73c0"
+      (reference "U?") (unit 1) (value "74LS08") (footprint "")
+    )
+    (path "/cc9b90a5-0c43-45c2-9570-29adffdd5447"
+      (reference "U?") (unit 1) (value "ATtiny84-20P") (footprint "Package_DIP:DIP-14_W7.62mm")
+    )
     (path "/ccd14c08-c4ab-4f62-97cd-05242c97da30"
       (reference "U?") (unit 1) (value "W65C22SxP") (footprint "")
     )
+    (path "/47e5f244-199c-483d-9129-db89de2f9ca8/cf5a01e8-a9be-4e84-9aa0-c1f4b57f7b20"
+      (reference "U?") (unit 1) (value "74LS02") (footprint "")
+    )
+    (path "/47e5f244-199c-483d-9129-db89de2f9ca8/cfc5aede-aaf1-484d-a71d-7fde6f5766b7"
+      (reference "U?") (unit 1) (value "CY62256-70PC") (footprint "Package_DIP:DIP-28_W15.24mm")
+    )
     (path "/d4ba973d-c535-4387-a638-737f289e743f"
       (reference "U?") (unit 1) (value "W65C02SxP") (footprint "Package_DIP:DIP-40_W15.24mm_Socket_LongPads")
     )
+    (path "/47e5f244-199c-483d-9129-db89de2f9ca8/16d92f16-835d-47cb-887c-c0a76290a59e"
+      (reference "U?") (unit 2) (value "74LS02") (footprint "")
+    )
     (path "/1a676615-df3c-4593-9789-3558c51cbded"
       (reference "U?") (unit 2) (value "74HC00") (footprint "")
     )
+    (path "/47e5f244-199c-483d-9129-db89de2f9ca8/392bf95e-a066-4f31-8ab9-03adeacb1ad1"
+      (reference "U?") (unit 2) (value "74HC00") (footprint "")
+    )
+    (path "/47e5f244-199c-483d-9129-db89de2f9ca8/9920babb-8886-48de-958d-96c19a7fc6e0"
+      (reference "U?") (unit 2) (value "74LS08") (footprint "")
+    )
+    (path "/47e5f244-199c-483d-9129-db89de2f9ca8/43ff5995-11bc-4eed-a78b-f2e9411b9686"
+      (reference "U?") (unit 3) (value "74LS08") (footprint "")
+    )
     (path "/98fa7777-1ce2-44a2-aa00-b0263af80f6b"
       (reference "U?") (unit 3) (value "74HC00") (footprint "")
     )
+    (path "/47e5f244-199c-483d-9129-db89de2f9ca8/b2b4b31b-3690-4b61-a4de-5607da02c81e"
+      (reference "U?") (unit 3) (value "74HC00") (footprint "")
+    )
+    (path "/47e5f244-199c-483d-9129-db89de2f9ca8/b3b777aa-d557-4e2d-92a8-84cf2fde425d"
+      (reference "U?") (unit 3) (value "74LS02") (footprint "")
+    )
+    (path "/47e5f244-199c-483d-9129-db89de2f9ca8/5b605d39-af40-4581-bff3-c2641732e6b0"
+      (reference "U?") (unit 4) (value "74HC00") (footprint "")
+    )
+    (path "/47e5f244-199c-483d-9129-db89de2f9ca8/6822bf7d-e2d9-40e8-8c53-382a10b80acb"
+      (reference "U?") (unit 4) (value "74LS08") (footprint "")
+    )
+    (path "/47e5f244-199c-483d-9129-db89de2f9ca8/81168c25-5bd6-4836-b1ca-2ad0d00544e1"
+      (reference "U?") (unit 4) (value "74LS02") (footprint "")
+    )
     (path "/dfa4aa66-61ba-424a-afda-7431ab2d5b3c"
       (reference "U?") (unit 4) (value "74HC00") (footprint "")
     )
+    (path "/47e5f244-199c-483d-9129-db89de2f9ca8/06bafd31-236f-42f3-afa3-5580a15f2ca0"
+      (reference "U?") (unit 5) (value "74LS08") (footprint "")
+    )
+    (path "/47e5f244-199c-483d-9129-db89de2f9ca8/28990dd7-74fd-483a-b8c4-f35cb4a11005"
+      (reference "U?") (unit 5) (value "74LS02") (footprint "")
+    )
     (path "/3a4de6b1-40ee-4ccf-b155-4fae4b0427a0"
       (reference "U?") (unit 5) (value "74HC00") (footprint "")
     )
+    (path "/47e5f244-199c-483d-9129-db89de2f9ca8/72e2621c-ca0e-4581-89aa-7a64ac107595"
+      (reference "U?") (unit 5) (value "74HC00") (footprint "")
+    )

Commit message: Finsing up peripherals almost done with schematic
Parts:
- removed C?: 0.1uF, symbol Device:C_Small
- removed R?: R_Small, symbol Device:R_Small
- removed U?: CY62256-70PC, Package_DIP:DIP-28_W15.24mm, symbol Memory_RAM:CY62256-70PC
- removed U?: 74LS245, Package_DIP:DIP-20_W7.62mm_Socket_LongPads, symbol 74xx:74LS245
- removed U?: 28C256, Package_DIP:DIP-28_W15.24mm_Socket_LongPads, symbol Memory_EEPROM:28C256
- removed U?: W65C22SxP, Package_DIP:DIP-40_W15.24mm_Socket_LongPads, symbol 65xx:W65C22SxP
- removed U?: ATtiny84-20P, Package_DIP:DIP-14_W7.62mm, symbol MCU_Microchip_ATtiny:ATtiny84-20P
- removed U?: W65C22SxP, symbol 65xx:W65C22SxP
- added C?: 0.1uF, symbol Device:C_Small
Connections:
- net +5V: now also C?.1, C?.1
- net GND: now also C?.2, C?.2
- net D0 renamed d0
- net D1 renamed d1
- net D2 renamed d2
- net D3 renamed d3
- net D4 renamed d4
- net D5 renamed d5
- net D6 renamed d6
- net D7 renamed d7
Other:
- added sheet IO (io.kicad_sch)
- moved on the sheet: C?, R?, U?A, U?E
