File: hardware/nevil_sbc_rev0/nevil_sbc_rev0.kicad_sch (KiCad schematic)
At the start: 27 parts, among them J101 Power, J102 Clock Selector, SW101 RESET, U101 74AC00, U102 NE555D, U103 74HC688, U104 W65C02SxP, X101 1MHz

Commit message: Working on pcb
Connections:
- net CLK: now also J102.2 (Pin_2); no longer J102.1 (Pin_1)
- net CLKOUT: now also J102.1 (Pin_1); no longer J102.2 (Pin_2)
Changed lines of the file:
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@@
     )
   )
-  (global_label "CLKOUT" (shape input) (at 43.815 139.7 0) (fields_autoplaced)
+  (global_label "CLK" (shape output) (at 43.815 139.7 0) (fields_autoplaced)
     (effects (font (size 1.27 1.27)) (justify left))
-    (property "Intersheet References" "${INTERSHEET_REFS}" (id 0) (at 53.4248 139.7794 0)
+    (property "Intersheet References" "${INTERSHEET_REFS}" (id 0) (at 49.7962 139.6206 0)
       (effects (font (size 1.27 1.27)) (justify left) hide)
     )
@@
     )
   )
-  (global_label "CLK" (shape output) (at 43.815 136.525 0) (fields_autoplaced)
+  (global_label "CLKOUT" (shape input) (at 43.815 136.525 0) (fields_autoplaced)
     (effects (font (size 1.27 1.27)) (justify left))
-    (property "Intersheet References" "${INTERSHEET_REFS}" (id 0) (at 49.7962 136.4456 0)
+    (property "Intersheet References" "${INTERSHEET_REFS}" (id 0) (at 53.4248 136.4456 0)
       (effects (font (size 1.27 1.27)) (justify left) hide)
     )

Commit message: working on vga code
Parts:
- added H101, H102, H104, H105: M3 Mounting Hole, MountingHole:MountingHole_3.2mm_M3_Pad, symbol Mechanical:MountingHole_Pad
- added H103: Expansion Support, MountingHole:MountingHole_3.2mm_M3_Pad, symbol Mechanical:MountingHole_Pad
Connections:
- net GND: now also H101.1, H102.1, H103.1, H104.1, H105.1
Other:
- note added: "Mounting Holes"
