File: hardware/nevil_sbc_rev0/peripherals.kicad_sch (KiCad schematic)
At the start: 24 parts

Commit message: Stashing work to switch machines
Parts:
- removed U? (x5): 74LS08, symbol 74xx:74LS08
- removed U? (x5): 74LS02, symbol 74xx:74LS02
- removed U? (x5): 74HC00, symbol 74xx:74HC00
- added U? (x7): 74LS04, symbol 74xx:74LS04
- added U? (x3): 74LS139, symbol 74xx:74LS139
Connections:
- net a4: now also U?.2 (A0)
- net a5: now also U?.3 (A1)
- net ~{IO}: now also U?.1; no longer U?.23 (~{CS2})
- net ~{VIA0}: now reaches U?.23 (~{CS2})
- net ~{VIA0}: now also U?.23 (~{CS2}), U?.4 (O0)
- net IO: now reaches U?.24 (CS1)
- net IO: now also U?.24 (CS1), U?.2
- new net GND: U?.1 (E)
- new net ~{EXT_IO}: U?.7 (O3)
- new net ~{PICO}: U?.6 (O2)
- new net ~{VIA1}: U?.5 (O1)
Other:
- note added: "IO: 0x8000...0x800F - VIA0 0x8010...0x801F - VIA1 0x8020...0x802F - PicoVGA 0x8030...0x803F - EXT_IO"
- note removed: "IO: 0x8000...0x800F - VIA0 0x8010...0x801F - VIA1 0X8020...0x803F - PicoVGA"
- moved on the sheet: U?

Commit message: Stashing work
Parts:
- U?: footprint (none) -> Package_DIP:DIP-16_W7.62mm_Socket_LongPads
Connections:
- net ~{VIA0}: no longer U?.23 (~{CS2})
- net ~{VIA1}: now also U?.23 (~{CS2})
- net v0pa3: now reaches U?.10 (PA3)
- net v0pa3: now also U?.5 (PA3)
- net v0pa2: now reaches U?.11 (PA2)
- net v0pa2: now also U?.4 (PA2)
- net v0pa1: now reaches U?.12 (PA1)
- net v0pa1: now also U?.3 (PA1)
- net v0pa0: now reaches U?.13 (AREF/PA0)
- net v0pa0: now also U?.2 (PA0)
- net v0pa8: now reaches U?.2 (XTAL1/PB0)
- net v0pa8: now also U?.40 (CA1)
- net KBDAT: now reaches U?.3 (XTAL2/PB1)
- net v0pa9: now reaches U?.4 (~{RESET}/PB3)
- net v0pa9: now also U?.39 (CA2)
- net KBCLK: now reaches U?.5 (PB2)
- net v0pa7: now reaches U?.6 (PA7)
- net v0pa7: now also U?.9 (PA7)
- net v0pa6: now reaches U?.7 (PA6)
- net v0pa6: now also U?.8 (PA6)
- net v0pa5: now reaches U?.8 (PA5)
- net v0pa5: now also U?.7 (PA5)
- net v0pa4: now reaches U?.9 (PA4)
- net v0pa4: now also U?.6 (PA4)
- net a3: now reaches U?.35 (RS3)
- net a2: now reaches U?.36 (RS2)
- net a1: now reaches U?.37 (RS1)
- net a0: now reaches U?.38 (RS0)
Other:
- moved on the sheet: U?

Commit message: Stashing work to continue on workstation
Parts:
- removed U?: W65C22SxP, symbol 65xx:W65C22SxP
- added C? (x6): 0.1uF, symbol Device:C_Small
- added U?: W65C22SxP, Package_DIP:DIP-40_W15.24mm_Socket_LongPads, symbol 65xx:W65C22SxP
- added U?: Pico, RPi_Pico:RPi_Pico_SMD_TH, symbol RPPico:Pico
Connections:
- net GND: now also U?.1 (VSS), U?.14 (GND), U?.14 (GND), U?.14 (GND), C?.2, C?.2, C?.2, C?.2, C?.2, C?.2, U?.1 (VSS)
- net IO: now also U?.24 (CS1)
- net KBCLK: now also U?.4 (~{RESET}/PB3); no longer U?.5 (PB2)
- net KBDAT: now also U?.5 (PB2); no longer U?.3 (XTAL2/PB1)
- net a0: now also U?.10 (A0), U?.10 (A0), U?.38 (RS0)
- net a1: now also U?.9 (A1), U?.9 (A1), U?.37 (RS1)
- net a2: now also U?.8 (A2), U?.8 (A2), U?.36 (RS2)
- net a3: now also U?.7 (A3), U?.7 (A3), U?.35 (RS3)
- net a4: now also U?.6 (A4), U?.6 (A4)
- net a5: now also U?.5 (A5), U?.5 (A5)
- net v0pa9: now also U?.3 (XTAL2/PB1); no longer U?.4 (~{RESET}/PB3)
- net ~{VIA1}: now also U?.23 (~{CS2})
- net a14: now reaches U?.1 (A14)
- net a14: now also U?.1 (A14)
- net d0: now reaches U?.11 (D0)
- net d0: now also U?.11 (Q0), U?.33 (D0), U?.33 (D0)
- net d1: now reaches U?.12 (D1)
- net d1: now also U?.12 (Q1), U?.32 (D1), U?.32 (D1)
- net d2: now reaches U?.13 (D2)
- net d2: now also U?.13 (Q2), U?.31 (D2), U?.31 (D2)
- net d3: now reaches U?.15 (D3)
- net d3: now also U?.15 (Q3), U?.30 (D3), U?.30 (D3)
- net d4: now reaches U?.16 (D4)
- net d4: now also U?.16 (Q4), U?.29 (D4), U?.29 (D4)
- net d5: now reaches U?.17 (D5)
- net d5: now also U?.17 (Q5), U?.28 (D5), U?.28 (D5)
- net d6: now reaches U?.18 (D6)
- net d6: now also U?.18 (Q6), U?.27 (D6), U?.27 (D6)
- net d7: now reaches U?.19 (D7)
- net d7: now also U?.19 (Q7), U?.26 (D7), U?.26 (D7)
- net a12: now reaches U?.2 (A12)
- net a12: now also U?.2 (A12)
- net ~{ROM}: now reaches U?.20 (~{CS})
- net a10: now reaches U?.21 (A10)
- net a10: now also U?.21 (A10)
- net ~{RD}: now reaches U?.22 (~{OE})
- net ~{RD}: now also U?.22 (~{OE})
- net a11: now reaches U?.23 (A11)
- net a11: now also U?.23 (A11)
- net a9: now reaches U?.24 (A9)
- net a9: now also U?.24 (A9)
- net a8: now reaches U?.25 (A8)
- net a8: now also U?.25 (A8)
- net a13: now reaches U?.26 (A13)
- net a13: now also U?.26 (A13)
- net ~{WR}: now reaches U?.27 (~{WE})
- net ~{WR}: now also U?.27 (~{WE})
- net +5V: now reaches U?.28 (VCC)
- net +5V: now also U?.1 (VCC), U?.20 (VCC), U?.28 (VCC), C?.1, C?.1, C?.1, C?.1, C?.1, C?.1, U?.20 (VCC)
- net a7: now reaches U?.3 (A7)
- net a7: now also U?.3 (A7)
- net a6: now reaches U?.4 (A6)
- net a6: now also U?.4 (A6)
- net v0pb0: now reaches U?.10 (PB0)
- net v0pb1: now reaches U?.11 (PB1)
- net v0pb2: now reaches U?.12 (PB2)
- net v0pb3: now reaches U?.13 (PB3)
- net v0pb4: now reaches U?.14 (PB4)
- net v0pb5: now reaches U?.15 (PB5)
- net v0pb6: now reaches U?.16 (PB6)
- net v0pb7: now reaches U?.17 (PB7)
- net ~{VIA0_IRQ}: now reaches U?.21 (~{IRQ})
- net R/~{W}: now reaches U?.22 (R/~{W})
- net R/~{W}: now also U?.22 (R/~{W})
- net CLK: now reaches U?.25 (ϕ2)
- net CLK: now also U?.25 (ϕ2)
- net ~{RESET}: now reaches U?.34 (~{RES})
- net ~{RESET}: now also U?.34 (~{RES})
- net ~{RAM}: now reaches U?.20 (~{CS})
- new net v1pa0: U?.2 (PA0)
- new net v1pa1: U?.3 (PA1)
- new net v1pa2: U?.4 (PA2)
- new net v1pa3: U?.5 (PA3)
- new net v1pa4: U?.6 (PA4)
- new net v1pa5: U?.7 (PA5)
- new net v1pa6: U?.8 (PA6)
- new net v1pa7: U?.9 (PA7)
- new net v1pa8: U?.40 (CA1)
- new net v1pa9: U?.39 (CA2)
- new net v1pb0: U?.10 (PB0)
- new net v1pb1: U?.11 (PB1)
- new net v1pb2: U?.12 (PB2)
- new net v1pb3: U?.13 (PB3)
- new net v1pb4: U?.14 (PB4)
- new net v1pb5: U?.15 (PB5)
- new net v1pb6: U?.16 (PB6)
- new net v1pb7: U?.17 (PB7)
- new net v1pb8: U?.18 (CB1)
- new net v1pb9: U?.19 (CB2)
- new net ~{VIA1_IRQ}: U?.21 (~{IRQ})
- no-connect marks 0 -> 2
Other:
- moved on the sheet: U?, U?B, U?C

Commit message: Finsing up peripherals almost done with schematic
Parts:
- removed C?: 0.1uF, symbol Device:C_Small
- removed C?: 1000uF, symbol Device:C_Polarized_Small
- removed R?: R_Small, symbol Device:R_Small
- removed U?: 74LS245, Package_DIP:DIP-20_W7.62mm_Socket_LongPads, symbol 74xx:74LS245
- removed U?: Pico, RPi_Pico:RPi_Pico_SMD_TH, symbol RPPico:Pico
- added C? (x3): 0.1uF, symbol Device:C_Small
- added U? (x5): 74LS08, symbol 74xx:74LS08
Connections:
- net +5V: now also U?.14 (VCC), U?.16 (VCC), C?.1, C?.1, C?.1, U?.14 (VCC)
- net GND: now also U?.7 (GND), U?.8 (GND), C?.2, C?.2, C?.2, U?.7 (GND); no longer U?.1 (E)
- net a6: now also U?.14 (A0)
- net a7: now also U?.13 (A1)
- net ~{IO}: now also U?.15 (E)
- net ~{VIA0_IRQ}: now also U?.1
- net ~{VIA1_IRQ}: now also U?.2
- net ~{EXT_IO2}: now reaches U?.10 (O2)
- net ~{EXT_IO1}: now reaches U?.11 (O1)
- net at U?.12 (O0): now also U?.1 (E)
- net ~{EXT_IO} renamed ~{EXT_IO0}
- new net: U?.3, U?.9
- new net: U?.10, U?.6
- new net ~{EXT_IO_IRQ}: U?.5
- new net ~{IRQ}: U?.8
- new net ~{PICO_IRQ}: U?.4
- no-connect marks 2 -> 16
Other:
- note added: "(and unused gates)"
- note added: "Atmega Keyboard logic"
- note added: "IO Address logic"
- note added: "IRQ Logic"
- note added: "Ram"
- note added: "Rom"
- note added: "Spare NOT gates"
- note added: "Via's"
- note added: "logic gates power supply"
- moved on the sheet: C?, U?A, U?B, U?C, U?D, U?E, U?F, U?G

Commit message: Finishing base schematic
Parts:
- removed C?: 0.1uF, symbol Device:C_Small
- added D201: V1PA7 LED, LED_THT:LED_D3.0mm, symbol Device:LED
- added R201: 1K, Resistor_THT:R_Axial_DIN0204_L3.6mm_D1.6mm_P7.62mm_Horizontal, symbol Device:R_Small
- C201, C202, C203, C205, C206, C207, C208, C209: renamed from C?; footprint (none) -> Capacitor_THT:C_Disc_D5.0mm_W2.5mm_P5.00mm
- U201: renamed from U?; value 74LS04 -> 74AC04; footprint (none) -> Package_DIP:DIP-14_W7.62mm_Socket_LongPads
- U202: renamed from U?; value 74LS139 -> 74AC139; footprint (none) -> Package_SO:TSSOP-14_4.4x5mm_P0.65mm
- U202: renamed from U?; value 74LS139 -> 74AC139; footprint Package_DIP:DIP-16_W7.62mm_Socket_LongPads -> Package_SO:TSSOP-14_4.4x5mm_P0.65mm
- U203: renamed from U?; value 74LS08 -> 74AC08; footprint (none) -> Package_DIP:DIP-14_W7.62mm_Socket_LongPads
- U204: renamed from U?; footprint Package_DIP:DIP-28_W15.24mm -> Package_DIP:DIP-28_W15.24mm_Socket_LongPads
- gave numbers to parts that had none: 4
Connections:
- net GND: now also R201.2
- net v0pb7: now also D201.2 (A)
- new net: D201.1 (K), R201.1
Other:
- note added: "V0PB7 Led."
- moved on the sheet: C206, U203C, U203D

Commit message: Add pcb files and small clk change for pico
Parts:
- U207: value W65C22SxP -> VIA0
- U208: value W65C22SxP -> VIA1
Connections:
- net CLK: now also U203.12
- net ~{PICO}: now also U201.3
- net PICO: now reaches U201.4
- net PICO: now also U203.13
- net PICO_CS_IN: now reaches U203.11
- no-connect marks 16 -> 11
Other:
- note added: "Pico CS Logic"
- moved on the sheet: U201A, U201B, U203D
Changed lines of the file:
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@@
   (no_connect (at 35.56 54.61))
   (no_connect (at 20.32 69.85))
-  (no_connect (at 35.56 22.86))
-  (no_connect (at 20.32 22.86))
   (no_connect (at 35.56 38.1))
   (no_connect (at 20.32 54.61))
@@
   (no_connect (at 20.32 84.455))
   (no_connect (at 157.48 53.975))
-  (no_connect (at 84.455 88.9))
-  (no_connect (at 84.455 83.82))
-  (no_connect (at 99.695 86.36))
   (no_connect (at 61.595 180.975))
   (no_connect (at 61.595 178.435))
@@
     (stroke (width 0) (type default) (color 0 0 0 0))
   )
+  (polyline (pts (xy 245.745 24.765) (xy 245.745 62.23))
+    (stroke (width 0) (type default) (color 0 0 0 0))
+  )
   (polyline (pts (xy 41.275 92.71) (xy 41.275 12.065))
     (stroke (width 0) (type default) (color 0 0 0 0))
@@
     (stroke (width 0) (type default) (color 0 0 0 0))
   )
-  (wire (pts (xy 168.91 42.545) (xy 170.18 42.545))
+  (wire (pts (xy 169.545 43.18) (xy 170.815 43.18))
     (stroke (width 0) (type default) (color 0 0 0 0))
   )
@@
     (stroke (width 0) (type default) (color 0 0 0 0))
   )
+  (polyline (pts (xy 196.215 24.765) (xy 245.745 24.765))
+    (stroke (width 0) (type default) (color 0 0 0 0))
+  )
   (wire (pts (xy 93.98 74.295) (xy 96.52 74.295))
     (stroke (width 0) (type default) (color 0 0 0 0))
@@
     (stroke (width 0) (type default) (color 0 0 0 0))
   )
+  (wire (pts (xy 224.155 48.895) (xy 226.695 48.895))
+    (stroke (width 0) (type default) (color 0 0 0 0))
+  )
   (bus (pts (xy 220.345 106.045) (xy 220.345 108.585))
     (stroke (width 0) (type default) (color 0 0 0 0))
@@
     (stroke (width 0) (type default) (color 0 0 0 0))
   )
-  (wire (pts (xy 185.42 42.545) (xy 186.69 42.545))
+  (wire (pts (xy 186.055 43.18) (xy 187.325 43.18))
     (stroke (width 0) (type default) (color 0 0 0 0))
   )
@@
     (stroke (width 0) (type default) (color 0 0 0 0))
   )
+  (wire (pts (xy 206.375 46.355) (xy 208.915 46.355))
+    (stroke (width 0) (type default) (color 0 0 0 0))
+  )
   (wire (pts (xy 122.555 158.115) (xy 130.175 158.115))
     (stroke (width 0) (type default) (color 0 0 0 0))
@@
     (stroke (width 0) (type default) (color 0 0 0 0))
   )
+  (wire (pts (xy 206.375 51.435) (xy 208.915 51.435))
+    (stroke (width 0) (type default) (color 0 0 0 0))
+  )
   (wire (pts (xy 189.23 123.825) (xy 194.31 123.825))
     (stroke (width 0) (type default) (color 0 0 0 0))
@@
     (stroke (width 0) (type default) (color 0 0 0 0))
   )
+  (wire (pts (xy 224.155 35.56) (xy 227.33 35.56))
+    (stroke (width 0) (type default) (color 0 0 0 0))
+  )
   (wire (pts (xy 28.575 145.415) (xy 31.115 145.415))
     (stroke (width 0) (type default) (color 0 0 0 0))
@@
     (stroke (width 0) (type default) (color 0 0 0 0))
   )
+  (wire (pts (xy 208.915 35.56) (xy 207.01 35.56))
+    (stroke (width 0) (type default) (color 0 0 0 0))
+  )
   (bus (pts (xy 273.685 114.935) (xy 273.685 117.475))
     (stroke (width 0) (type default) (color 0 0 0 0))
@@
     (stroke (width 0) (type default) (color 0 0 0 0))
   )
+  (polyline (pts (xy 245.745 62.23) (xy 196.215 62.23))
+    (stroke (width 0) (type default) (color 0 0 0 0))
+  )
   (bus (pts (xy 124.46 46.99) (xy 125.095 46.99))
     (stroke (width 0) (type default) (color 0 0 0 0))
@@
     (effects (font (size 1.27 1.27)) (justify left bottom))
   )
+  (text "Pico CS Logic" (at 230.505 60.96 0)
+    (effects (font (size 1.27 1.27) italic) (justify left bottom))
+  )
   (text "V0PB7 Led." (at 139.065 196.85 0)
     (effects (font (size 1.27 1.27)) (justify left bottom))
@@
     (effects (font (size 1.27 1.27)) (justify left bottom))
   )
-  (global_label "IO" (shape input) (at 186.69 42.545 0) (fields_autoplaced)
+  (global_label "IO" (shape input) (at 187.325 43.18 0) (fields_autoplaced)
     (effects (font (size 1.27 1.27)) (justify left))
-    (property "Intersheet References" "${INTERSHEET_REFS}" (id 0) (at 191.0383 42.4656 0)
+    (property "Intersheet References" "${INTERSHEET_REFS}" (id 0) (at 191.6733 43.1006 0)
+      (effects (font (size 1.27 1.27)) (justify left) hide)
+    )
+  )
+  (global_label "PICO_CS_IN" (shape input) (at 226.695 48.895 0) (fields_autoplaced)
+    (effects (font (size 1.27 1.27)) (justify left))
+    (property "Intersheet References" "${INTERSHEET_REFS}" (id 0) (at 239.9333 48.8156 0)
       (effects (font (size 1.27 1.27)) (justify left) hide)
     )
@@
     )
   )
+  (global_label "CLK" (shape input) (at 206.375 46.355 180) (fields_autoplaced)
+    (effects (font (size 1.27 1.27)) (justify right))
+    (property "Intersheet References" "${INTERSHEET_REFS}" (id 0) (at 200.3938 46.2756 0)
+      (effects (font (size 1.27 1.27)) (justify right) hide)
+    )
+  )
   (global_label "~{ROM}" (shape input) (at 191.135 158.115 180) (fields_autoplaced)
     (effects (font (size 1.27 1.27)) (justify right))
@@
     )
   )
-  (global_label "~{IO}" (shape input) (at 168.91 42.545 180) (fields_autoplaced)
+  (global_label "~{IO}" (shape input) (at 169.545 43.18 180) (fields_autoplaced)
     (effects (font (size 1.27 1.27)) (justify right))
-    (property "Intersheet References" "${INTERSHEET_REFS}" (id 0) (at 164.5617 42.4656 0)
+    (property "Intersheet References" "${INTERSHEET_REFS}" (id 0) (at 165.1967 43.1006 0)
       (effects (font (size 1.27 1.27)) (justify right) hide)
     )
@@
     )
   )
+  (global_label "PICO" (shape input) (at 206.375 51.435 180) (fields_autoplaced)
+    (effects (font (size 1.27 1.27)) (justify right))
+    (property "Intersheet References" "${INTERSHEET_REFS}" (id 0) (at 199.4867 51.5144 0)
+      (effects (font (size 1.27 1.27)) (justify right) hide)
+    )
+  )
   (global_label "~{RESET}" (shape input) (at 24.765 125.095 180) (fields_autoplaced)
     (effects (font (size 1.27 1.27)) (justify right))
@@
     )
   )
+  (global_label "PICO" (shape output) (at 227.33 35.56 0) (fields_autoplaced)
+    (effects (font (size 1.27 1.27)) (justify left))
+    (property "Intersheet References" "${INTERSHEET_REFS}" (id 0) (at 234.2183 35.4806 0)
+      (effects (font (size 1.27 1.27)) (justify left) hide)
+    )
+  )
   (global_label "~{VIA1}" (shape output) (at 168.91 26.67 0) (fields_autoplaced)
     (effects (font (size 1.27 1.27)) (justify left))
@@
     )
   )
+  (global_label "~{PICO}" (shape input) (at 207.01 35.56 180) (fields_autoplaced)
+    (effects (font (size 1.27 1.27)) (justify right))
+    (property "Intersheet References" "${INTERSHEET_REFS}" (id 0) (at 200.1217 35.4806 0)
+      (effects (font (size 1.27 1.27)) (justify right) hide)
+    )
+  )
   (global_label "~{VIA0_IRQ}" (shape input) (at 54.61 69.215 180) (fields_autoplaced)
     (effects (font (size 1.27 1.27)) (justify right))
@@
     (pin "1")
   )
-  (symbol (lib_id "74xx:74LS04") (at 27.94 22.86 0) (unit 2)
+  (symbol (lib_id "74xx:74LS04") (at 216.535 35.56 0) (unit 2)
     (in_bom yes) (on_board yes)
-    (property "Reference" "U201" (id 0) (at 27.94 15.875 0))
-    (property "Value" "74AC04" (id 1) (at 27.94 17.78 0))
-    (property "Footprint" "Package_DIP:DIP-14_W7.62mm_Socket_LongPads" (id 2) (at 27.94 22.86 0)
+    (property "Reference" "U201" (id 0) (at 216.535 28.575 0))
+    (property "Value" "74AC04" (id 1) (at 216.535 30.48 0))
+    (property "Footprint" "Package_DIP:DIP-14_W7.62mm_Socket_LongPads" (id 2) (at 216.535 35.56 0)
       (effects (font (size 1.27 1.27)) hide)
     )
-    (property "Datasheet" "http://www.ti.com/lit/gpn/sn74LS04" (id 3) (at 27.94 22.86 0)
+    (property "Datasheet" "http://www.ti.com/lit/gpn/sn74LS04" (id 3) (at 216.535 35.56 0)
       (effects (font (size 1.27 1.27)) hide)
     )
@@
       (effects (font (size 1.27 1.27)) (justify left))
     )
-    (property "Value" "W65C22SxP" (id 1) (at 109.3344 118.745 0)
+    (property "Value" "VIA1" (id 1) (at 109.3344 118.745 0)
       (effects (font (size 1.27 1.27) bold italic) (justify left))
     )
@@
       (effects (font (size 1.27 1.27)) (justify left))
     )
-    (property "Value" "W65C22SxP" (id 1) (at 48.3744 118.745 0)
+    (property "Value" "VIA0" (id 1) (at 48.3744 118.745 0)
       (effects (font (size 1.27 1.27) bold italic) (justify left))
     )
@@
     (pin "1")
   )
-  (symbol (lib_id "74xx:74LS04") (at 177.8 42.545 0) (unit 1)
+  (symbol (lib_id "74xx:74LS04") (at 178.435 43.18 0) (unit 1)
     (in_bom yes) (on_board yes)
-    (property "Reference" "U201" (id 0) (at 177.8 34.29 0))
-    (property "Value" "74AC04" (id 1) (at 177.8 36.83 0))
-    (property "Footprint" "Package_DIP:DIP-14_W7.62mm_Socket_LongPads" (id 2) (at 177.8 42.545 0)
+    (property "Reference" "U201" (id 0) (at 178.435 34.925 0))
+    (property "Value" "74AC04" (id 1) (at 178.435 37.465 0))
+    (property "Footprint" "Package_DIP:DIP-14_W7.62mm_Socket_LongPads" (id 2) (at 178.435 43.18 0)
       (effects (font (size 1.27 1.27)) hide)
     )
-    (property "Datasheet" "http://www.ti.com/lit/gpn/sn74LS04" (id 3) (at 177.8 42.545 0)
+    (property "Datasheet" "http://www.ti.com/lit/gpn/sn74LS04" (id 3) (at 178.435 43.18 0)
       (effects (font (size 1.27 1.27)) hide)
     )
@@
     (pin "9")
   )
-  (symbol (lib_id "74xx:74LS08") (at 92.075 86.36 0) (unit 4)
+  (symbol (lib_id "74xx:74LS08") (at 216.535 48.895 0) (unit 4)
     (in_bom yes) (on_board yes)
-    (property "Reference" "U203" (id 0) (at 92.075 79.375 0))
-    (property "Value" "74AC08" (id 1) (at 92.075 81.28 0))
-    (property "Footprint" "Package_DIP:DIP-14_W7.62mm_Socket_LongPads" (id 2) (at 92.075 86.36 0)
+    (property "Reference" "U203" (id 0) (at 216.535 41.91 0))
+    (property "Value" "74AC08" (id 1) (at 216.535 43.815 0))
+    (property "Footprint" "Package_DIP:DIP-14_W7.62mm_Socket_LongPads" (id 2) (at 216.535 48.895 0)
       (effects (font (size 1.27 1.27)) hide)
     )
-    (property "Datasheet" "http://www.ti.com/lit/gpn/sn74LS08" (id 3) (at 92.075 86.36 0)
+    (property "Datasheet" "http://www.ti.com/lit/gpn/sn74LS08" (id 3) (at 216.535 48.895 0)
       (effects (font (size 1.27 1.27)) hide)
     )

Commit message: working on vga code
Parts:
- U202: footprint Package_SO:TSSOP-14_4.4x5mm_P0.65mm -> Package_SO:TSSOP-16_4.4x5mm_P0.65mm
Other:
- note added: "IO: 0x8000...0x800F - VIA0 0x8010...0x801F - VIA1 0x8020...0x802F - PicoVGA 0x8030...0x803F - EXT_IO_0 0x8040...0x804F - EXT_IO_1 0x8050...0x805F - EXT_IO_2"
- note removed: "IO: 0x8000...0x800F - VIA0 0x8010...0x801F - VIA1 0x8020...0x802F - PicoVGA 0x8030...0x803F - EXT_IO"
Changed lines of the file:
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@@
     (effects (font (size 1.27 1.27)) (justify left bottom))
   )
-  (text "IO:\n0x8000...0x800F - VIA0\n0x8010...0x801F - VIA1\n0x8020...0x802F - PicoVGA\n0x8030...0x803F - EXT_IO\n"
-    (at 256.54 23.495 0)
+  (text "IO:\n0x8000...0x800F - VIA0\n0x8010...0x801F - VIA1\n0x8020...0x802F - PicoVGA\n0x8030...0x803F - EXT_IO_0\n0x8040...0x804F - EXT_IO_1\n0x8050...0x805F - EXT_IO_2\n"
+    (at 255.905 27.94 0)
     (effects (font (size 1.27 1.27)) (justify left bottom))
   )
@@
     (property "Reference" "U202" (id 0) (at 144.78 40.005 0))
     (property "Value" "74AC139" (id 1) (at 144.78 42.545 0))
-    (property "Footprint" "Package_SO:TSSOP-14_4.4x5mm_P0.65mm" (id 2) (at 144.78 48.895 0)
+    (property "Footprint" "Package_SO:TSSOP-16_4.4x5mm_P0.65mm" (id 2) (at 144.78 48.895 0)
       (effects (font (size 1.27 1.27)) hide)
     )
@@
       (effects (font (size 1.27 1.27)) (justify left))
     )
-    (property "Footprint" "Package_SO:TSSOP-14_4.4x5mm_P0.65mm" (id 2) (at 83.82 36.83 0)
+    (property "Footprint" "Package_SO:TSSOP-16_4.4x5mm_P0.65mm" (id 2) (at 83.82 36.83 0)
       (effects (font (size 1.27 1.27)) hide)
     )
@@
     (property "Reference" "U202" (id 0) (at 145.415 17.78 0))
     (property "Value" "74AC139" (id 1) (at 144.78 20.32 0))
-    (property "Footprint" "Package_SO:TSSOP-14_4.4x5mm_P0.65mm" (id 2) (at 145.415 26.67 0)
-      (effects (font (size 1.27 1.27)) hide)
-    )
+    (property "Footprint" "Package_SO:TSSOP-16_4.4x5mm_P0.65mm" (id 2) (at 145.415 26.67 0)
+      (effects (font (size 1.27 1.27)) hide)
+    )
